File: pcb/U3A_rs485.kicad_sch (KiCad schematic)
At the start: 18 parts, among them J1 Screw_Terminal_01x06, J2 Conn_01x07_Socket, J3 Conn_01x02_Pin, J4 Conn_01x08_Socket, J5 Conn_01x02_Pin, U1 THVD1452DR

Commit message: Change vendor of parts
Parts:
- H1, H2: Vendor HTL, DigiKey -> HTL; VendorId 100991, 100993, 732-12987-ND -> 100991, 100993, 103622
- J1: Vendor DigiKey -> HTL; VendorId 277-1724-ND -> 103639
- U1: Vendor DigiKey -> HTL; VendorId 296-THVD1452DRCT-ND -> 103640
Changed lines of the file:
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@@
       (effects (font (size 1.27 1.27)) hide)
     )
-    (property "Vendor" "HTL, DigiKey" (at 215.9 151.13 0)
-      (effects (font (size 1.27 1.27)) hide)
-    )
-    (property "VendorId" "100991, 100993, 732-12987-ND" (at 215.9 151.13 0)
+    (property "Vendor" "HTL" (at 215.9 151.13 0)
+      (effects (font (size 1.27 1.27)) hide)
+    )
+    (property "VendorId" "100991, 100993, 103622" (at 215.9 151.13 0)
       (effects (font (size 1.27 1.27)) hide)
     )
@@
       (effects (font (size 1.27 1.27)) hide)
     )
-    (property "Vendor" "DigiKey" (at 185.42 85.09 0)
-      (effects (font (size 1.27 1.27)) hide)
-    )
-    (property "VendorId" "277-1724-ND" (at 185.42 85.09 0)
+    (property "Vendor" "HTL" (at 185.42 85.09 0)
+      (effects (font (size 1.27 1.27)) hide)
+    )
+    (property "VendorId" "103639" (at 185.42 85.09 0)
       (effects (font (size 1.27 1.27)) hide)
     )
@@
       (effects (font (size 1.27 1.27)) hide)
     )
-    (property "Vendor" "HTL, DigiKey" (at 205.74 151.13 0)
-      (effects (font (size 1.27 1.27)) hide)
-    )
-    (property "VendorId" "100991, 100993, 732-12987-ND" (at 205.74 151.13 0)
+    (property "Vendor" "HTL" (at 205.74 151.13 0)
+      (effects (font (size 1.27 1.27)) hide)
+    )
+    (property "VendorId" "100991, 100993, 103622" (at 205.74 151.13 0)
       (effects (font (size 1.27 1.27)) hide)
     )
@@
       (effects (font (size 1.27 1.27) italic) hide)
     )
-    (property "Vendor" "DigiKey" (at 139.7 83.82 0)
-      (effects (font (size 1.27 1.27)) hide)
-    )
-    (property "VendorId" "296-THVD1452DRCT-ND" (at 139.7 83.82 0)
-      (effects (font (size 1.27 1.27)) hide)
-    )
+    (property "Vendor" "HTL" (at 139.7 83.82 0)
+      (effects (font (size 1.27 1.27)) hide)
+    )
+    (property "VendorId" "103640" (at 139.7 83.82 0)
+      (effects (font (size 1.27 1.27)) hide)
+    )

Commit message: Update to KiCAD 9
Parts:
- FID1, FID2, FID3, FID4, H1, H2: now left out of the parts list

Commit message: Rename/Add/Remove bom fields
Parts:
- C1, C2: HTL (none) -> 100140; Vendor HTL -> (none); VendorId 100140 -> (none)
- C3: HTL (none) -> 100128; Vendor HTL -> (none); VendorId 100128 -> (none)
- H1, H2: HTL (none) -> 100991, 100993, 103622; Vendor HTL -> (none); VendorId 100991, 100993, 103622 -> (none)
- J1: HTL (none) -> 103639; Vendor HTL -> (none); VendorId 103639 -> (none)
- J2, J4: HTL (none) -> 101546; Vendor HTL -> (none); VendorId 101546 -> (none)
- J3, J5: HTL (none) -> 101521; Vendor HTL -> (none); VendorId 101521 -> (none)
- R1, R2: HTL (none) -> 102933; Vendor HTL -> (none); VendorId 102933 -> (none)
- R3: HTL (none) -> 102967; Vendor HTL -> (none); VendorId 102967 -> (none)
- U1: HTL (none) -> 103640; Vendor HTL -> (none); VendorId 103640 -> (none)
Changed lines of the file:
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@@
 			)
 		)
-		(property "Vendor" "HTL"
-			(at 114.3 106.68 0)
-			(effects
-				(font
-					(size 1.27 1.27)
-				)
-				(hide yes)
-			)
-		)
-		(property "VendorId" "102967"
-			(at 114.3 106.68 0)
+		(property "HTL" "102967"
+			(at 114.3 106.68 90)
 			(effects
 				(font
@@
 			)
 		)
-		(property "Vendor" "HTL"
-			(at 215.9 151.13 0)
-			(effects
-				(font
-					(size 1.27 1.27)
-				)
-				(hide yes)
-			)
-		)
-		(property "VendorId" "100991, 100993, 103622"
-			(at 215.9 151.13 0)
+		(property "HTL" "100991, 100993, 103622"
+			(at 215.9 151.13 90)
 			(effects
 				(font
@@
 			)
 		)
-		(property "Vendor" "HTL"
-			(at 161.29 96.52 0)
-			(effects
-				(font
-					(size 1.27 1.27)
-				)
-				(hide yes)
-			)
-		)
-		(property "VendorId" "102933"
-			(at 161.29 96.52 0)
+		(property "HTL" "102933"
+			(at 161.29 96.52 90)
 			(effects
 				(font
@@
 		)
 		(property "Description" "Fiducial Marker"
-			(at 254 152.4 0)
-			(effects
-				(font
-					(size 1.27 1.27)
-				)
-				(hide yes)
-			)
-		)
-		(property "Vendor" ""
-			(at 254 152.4 0)
-			(effects
-				(font
-					(size 1.27 1.27)
-				)
-				(hide yes)
-			)
-		)
-		(property "VendorId" ""
 			(at 254 152.4 0)
 			(effects
@@
 			)
 		)
-		(property "Vendor" "HTL"
-			(at 171.45 71.12 0)
-			(effects
-				(font
-					(size 1.27 1.27)
-				)
-				(hide yes)
-			)
-		)
-		(property "VendorId" "101521"
+		(property "HTL" "101521"
 			(at 171.45 71.12 0)
 			(effects
@@
 			)
 		)
-		(property "Vendor" "HTL"
-			(at 185.42 85.09 0)
-			(effects
-				(font
-					(size 1.27 1.27)
-				)
-				(hide yes)
-			)
-		)
-		(property "VendorId" "103639"
+		(property "HTL" "103639"
 			(at 185.42 85.09 0)
 			(effects
@@
 			)
 		)
-		(property "Vendor" ""
-			(at 228.6 152.4 0)
-			(effects
-				(font
-					(size 1.27 1.27)
-				)
-				(hide yes)
-			)
-		)
-		(property "VendorId" ""
-			(at 228.6 152.4 0)
-			(effects
-				(font
-					(size 1.27 1.27)
-				)
-				(hide yes)
-			)
-		)
 		(instances
 			(project "U3A_rs485"
@@
 		)
 		(property "Description" "Fiducial Marker"
-			(at 266.7 152.4 0)
-			(effects
-				(font
-					(size 1.27 1.27)
-				)
-				(hide yes)
-			)
-		)
-		(property "Vendor" ""
-			(at 266.7 152.4 0)
-			(effects
-				(font
-					(size 1.27 1.27)
-				)
-				(hide yes)
-			)
-		)
-		(property "VendorId" ""
 			(at 266.7 152.4 0)
 			(effects
@@
 			)
 		)
-		(property "Vendor" "HTL"
-			(at 101.6 177.8 0)
-			(effects
-				(font
-					(size 1.27 1.27)
-				)
-				(hide yes)
-			)
-		)
-		(property "VendorId" "100140"
+		(property "HTL" "100140"
 			(at 101.6 177.8 0)
 			(effects
@@
 			)
 		)
-		(property "Vendor" "HTL"
-			(at 114.3 177.8 0)
-			(effects
-				(font
-					(size 1.27 1.27)
-				)
-				(hide yes)
-			)
-		)
-		(property "VendorId" "100140"
+		(property "HTL" "100140"
 			(at 114.3 177.8 0)
 			(effects
@@
 		)
 		(property "Description" "Fiducial Marker"
-			(at 241.3 152.4 0)
-			(effects
-				(font
-					(size 1.27 1.27)
-				)
-				(hide yes)
-			)
-		)
-		(property "Vendor" ""
-			(at 241.3 152.4 0)
-			(effects
-				(font
-					(size 1.27 1.27)
-				)
-				(hide yes)
-			)
-		)
-		(property "VendorId" ""
 			(at 241.3 152.4 0)
 			(effects
@@
 			)
 		)
-		(property "Vendor" "HTL"
-			(at 171.45 96.52 0)
-			(effects
-				(font
-					(size 1.27 1.27)
-				)
-				(hide yes)
-			)
-		)
-		(property "VendorId" "101521"
+		(property "HTL" "101521"
 			(at 171.45 96.52 0)
 			(effects
@@
 			)
 		)
-		(property "Vendor" "HTL"
-			(at 205.74 151.13 0)
-			(effects
-				(font
-					(size 1.27 1.27)
-				)
-				(hide yes)
-			)
-		)
-		(property "VendorId" "100991, 100993, 103622"
-			(at 205.74 151.13 0)
+		(property "HTL" "100991, 100993, 103622"
+			(at 205.74 151.13 90)
 			(effects
 				(font
@@
 			)
 		)
-		(property "Vendor" "HTL"
-			(at 127 177.8 0)
-			(effects
-				(font
-					(size 1.27 1.27)
-				)
-				(hide yes)
-			)
-		)
-		(property "VendorId" "100128"
+		(property "HTL" "100128"
 			(at 127 177.8 0)
 			(effects
@@
 			)
 		)
-		(property "Vendor" "HTL"
-			(at 161.29 71.12 0)
-			(effects
-				(font
-					(size 1.27 1.27)
-				)
-				(hide yes)
-			)
-		)
-		(property "VendorId" "102933"
-			(at 161.29 71.12 0)
+		(property "HTL" "102933"
+			(at 161.29 71.12 90)
 			(effects
 				(font
@@
 			)
 		)
-		(property "Vendor" "HTL"
-			(at 124.46 129.54 0)
-			(effects
-				(font
-					(size 1.27 1.27)
-				)
-				(hide yes)
-			)
-		)
-		(property "VendorId" "101546"
-			(at 124.46 129.54 0)
+		(property "HTL" "101546"
+			(at 124.46 129.54 90)
 			(effects
 				(font
@@
 			)
 		)
-		(property "Vendor" "HTL"
-			(at 97.79 90.17 0)
-			(effects
-				(font
-					(size 1.27 1.27)
-				)
-				(hide yes)
-			)
-		)
-		(property "VendorId" "101546"
-			(at 97.79 90.17 0)
+		(property "HTL" "101546"
+			(at 97.79 90.17 90)
 			(effects
 				(font
@@
 			)
 		)
-		(property "Vendor" "HTL"
+		(property "HTL" "103640"
 			(at 139.7 83.82 0)
 			(effects
-				(font
-					(size 1.27 1.27)
-				)
-				(hide yes)
-			)
-		)
-		(property "VendorId" "103640"
-			(at 139.7 83.82 0)
-			(effects
